File: board/TinyFPGA-A-Programmer.kicad_pcb (KiCad board)
At the start: 2 copper layers, 17.8 x 27.9 mm, 9 parts, among them J1 USB, J2 JTAG, J3 ICSP, U1 PIC16F1455-QFN16, U2 MIC5504-3.3YM5-TR

Commit message: updated schematic and PCB
Parts:
- added D+: TEST, Measurement_Points:Measurement_Point_Round-SMD-Pad_Small, B.Cu at (145.9, 106.9)
- added D-: TEST, Measurement_Points:Measurement_Point_Round-SMD-Pad_Small, B.Cu at (149.5, 106.8)
- added J2: JTAG, TinyFPGA:Pin_Header_Straight_1x05_Pitch2.54mm_SMD, F.Cu at (147.3, 119.4)
- added J2: JTAG, Pin_Headers:Pin_Header_Straight_1x05_Pitch2.54mm, F.Cu at (142.2, 126.9)
- added J2: JTAG, Pin_Headers:Pin_Header_Straight_1x05_Pitch2.54mm, F.Cu at (142.2, 129.4)
- added J4: CONN_01X06, Pin_Headers:Pin_Header_Straight_1x06_Pitch2.54mm, F.Cu at (154.9, 104.1)
- added REF***: OSHW-Logo_5.7x6mm_SilkScreen, Symbols:OSHW-Logo_5.7x6mm_SilkScreen, B.Cu at (147.7, 111.0)
- added VUSB: TEST, Measurement_Points:Measurement_Point_Round-SMD-Pad_Small, B.Cu at (147.7, 102.5)
- moved C1 4.52 mm to (151.0, 110.7), turned to 180 degrees
- moved C4 3.51 mm to (148.1, 115.7)
- moved C2 2.73 mm to (151.0, 116.4), turned to 180 degrees
- moved C3 2.57 mm to (144.6, 111.0)
- moved U1 2.57 mm to (144.6, 114.9)
- moved J2 2.54 mm to (142.2, 124.5)
- moved U2 1.77 mm to (150.8, 113.8)
Connections:
- U1 pad 1: Net-(U1-Pad1) -> RA5
- U1 pad 2: Net-(U1-Pad2) -> RA4
Routing:
- net GND: track 8.24 -> 101.2 mm, vias 6 -> 31
- net RA5: track 0.00 -> 17.3 mm, vias 0 -> 2
- net RA4: track 0.00 -> 13.8 mm, vias 0 -> 1
- net ICSPCLK: track 7.17 -> 17.4 mm
- net ICSPDAT: track 7.54 -> 17.0 mm, vias 1 -> 2
- net +3V3: track 19.3 -> 27.7 mm
- net Net-(J2-Pad5): track 11.1 -> 19.3 mm
- net +5V: track 14.8 -> 21.6 mm, vias 0 -> 1
- net Net-(J2-Pad3): track 9.31 -> 15.8 mm, vias 0 -> 2
- net Net-(J2-Pad2): track 8.06 -> 13.9 mm
- net Net-(J2-Pad1): track 8.70 -> 13.6 mm
- net VPP: track 11.1 -> 8.59 mm
- net Net-(J1-Pad2): track 13.6 -> 13.0 mm, vias 0 -> 1
- net Net-(J1-Pad3): track 12.7 -> 12.1 mm, vias 0 -> 1
Other:
- board size 17.8 x 27.9 mm -> 17.8 x 30.5 mm
- board text added: ".125"
- board text added: ".150"
- board text added: ".175"
- board text added: "3v3"
- board text added: "RA4"
- board text added: "RA5"
- board text added: "RC0"
- board text added: "RC1"
- board text added: "RC2/TDO"
- board text added: "RC3/TDI"
- board text added: "RC4/TCK"
- board text added: "RC5/TMS"
